File: KiCad Files/GeoSence_KiCad single module/GeoSence_KiCad_singal_module/GeoSence_KiCad_singal_module.kicad_pcb (KiCad board)
At the start: 2 copper layers, 50 x 30 mm, 26 parts, among them J1 Thermistor input, J2 Jumper pins, J3 Power Input, J4 Output Pins, J5 Conn_01x01_Socket, J6 Conn_01x01_Socket, J7 Conn_01x01_Socket, J8 Conn_01x01_Socket, U1 LM334Z, U2 LM334Z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

Commit message: updated to kicad 9.0.1
Other:
- board text added: "+5"
- board text added: "GND"
- board text added: "Input"
- board text added: "Output"
- board text added: "Testing and validation board"
