File: KiCad Files/GeoSence_KiCad single module/GeoSence_KiCad_singal_module/GeoSence_KiCad_singal_module.kicad_sch (KiCad schematic)
At the start: 26 parts, among them J1 Thermistor input, J2 Jumper pins, J3 Power Input, J4 Output Pins, J5 Conn_01x01_Socket, J6 Conn_01x01_Socket, J7 Conn_01x01_Socket, J8 Conn_01x01_Socket, U1 LM334Z, U2 LM334Z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

Commit message: updated to kicad 9.0.1
Other:
- note added: "Instrumentation amp Circuit"
- note removed: "Integrator Circuit"
Changed lines of the file:
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@@
 (kicad_sch
-	(version 20231120)
+	(version 20250114)
 	(generator "eeschema")
-	(generator_version "8.0")
+	(generator_version "9.0")
 	(paper "A5")
 	(title_block
@@
 		(rev "1")
 	)
+	(text "Reference Resistor supply"
+		(exclude_from_sim no)
+		(at 68.834 59.436 0)
+		(effects
+			(font
+				(size 1.27 1.27)
+			)
+		)
+	)
+	(text "Thermistor supply"
+		(exclude_from_sim no)
+		(at 21.082 59.182 0)
+		(effects
+			(font
+				(size 1.27 1.27)
+			)
+		)
+	)
+	(text "Thermistor input"
+		(exclude_from_sim no)
+		(at 20.574 82.55 0)
+		(effects
+			(font
+				(size 1.27 1.27)
+			)
+		)
+	)
+	(text "Output Pins"
+		(exclude_from_sim no)
+		(at 93.98 63.246 0)
+		(effects
+			(font
+				(size 1.27 1.27)
+			)
+		)
+	)
+	(text "Power input"
+		(exclude_from_sim no)
+		(at 61.214 82.296 0)
+		(effects
+			(font
+				(size 1.27 1.27)
+			)
+		)
+	)
+	(text "Instrumentation amp Circuit\n"
+		(exclude_from_sim no)
+		(at 105.918 14.224 0)
+		(effects
+			(font
+				(size 1.27 1.27)
+			)
+		)
+	)
+	(text "Not used"
+		(exclude_from_sim no)
+		(at 189.484 25.4 0)
+		(effects
+			(font
+				(size 1.27 1.27)
+			)
+		)
+	)
+	(text "Screw Holes"
+		(exclude_from_sim no)
+		(at 122.174 63.246 0)
+		(effects
+			(font
+				(size 1.27 1.27)
+			)
+		)
+	)
+	(text "Integrator circuit input"
+		(exclude_from_sim no)
+		(at 24.638 14.224 0)
+		(effects
+			(font
+				(size 1.27 1.27)
+			)
+		)
+	)
+	(text "Input Pins"
+		(exclude_from_sim no)
+		(at 17.78 62.23 0)
+		(effects
+			(font
+				(size 1.27 1.27)
+			)
+		)
+	)
 	(junction
 		(at 128.27 71.12)
@@
 		)
 	)
-	(text "Reference Resistor supply"
-		(exclude_from_sim no)
-		(at 68.834 59.436 0)
-		(effects
-			(font
-				(size 1.27 1.27)
-			)
-		)
-	)
-	(text "Thermistor supply"
-		(exclude_from_sim no)
-		(at 21.082 59.182 0)
-		(effects
-			(font
-				(size 1.27 1.27)
-			)
-		)
-	)
-	(text "Thermistor input"
-		(exclude_from_sim no)
-		(at 20.574 82.55 0)
-		(effects
-			(font
-				(size 1.27 1.27)
-			)
-		)
-	)
-	(text "Output Pins"
-		(exclude_from_sim no)
-		(at 93.98 63.246 0)
-		(effects
-			(font
-				(size 1.27 1.27)
-			)
-		)
-	)
-	(text "Power input"
-		(exclude_from_sim no)
-		(at 61.214 82.296 0)
-		(effects
-			(font
-				(size 1.27 1.27)
-			)
-		)
-	)
-	(text "Integrator Circuit"
-		(exclude_from_sim no)
-		(at 131.826 14.478 0)
-		(effects
-			(font
-				(size 1.27 1.27)
-			)
-		)
-	)
-	(text "Not used"
-		(exclude_from_sim no)
-		(at 189.484 25.4 0)
-		(effects
-			(font
-				(size 1.27 1.27)
-			)
-		)
-	)
-	(text "Screw Holes"
-		(exclude_from_sim no)
-		(at 122.174 63.246 0)
-		(effects
-			(font
-				(size 1.27 1.27)
-			)
-		)
-	)
-	(text "Integrator circuit input"
-		(exclude_from_sim no)
-		(at 24.638 14.224 0)
-		(effects
-			(font
-				(size 1.27 1.27)
-			)
-		)
-	)
-	(text "Input Pins"
-		(exclude_from_sim no)
-		(at 17.78 62.23 0)
-		(effects
-			(font
-				(size 1.27 1.27)
-			)
-		)
-	)
 	(global_label "Thermistor-in_1"
 		(shape input)
@@
 	)
 	(symbol
+		(lib_id "GeoSense logo G:LOGO")
+		(at 170.18 81.28 0)
+		(unit 1)
+		(exclude_from_sim no)
+		(in_bom yes)
+		(on_board yes)
+		(dnp no)
+		(fields_autoplaced yes)
+		(property "Reference" "#G1"
+			(at 170.18 62.7803 0)
+			(effects
+				(font
+					(size 1.27 1.27)
+				)
+				(hide yes)
+			)
+		)
+		(property "Value" "LOGO"
+			(at 170.18 99.7797 0)
+			(effects
+				(font
+					(size 1.27 1.27)
+				)
+				(hide yes)
+			)
+		)
+		(property "Footprint" "Logo kicad:GeoSenseGLogo"
+			(at 170.18 81.28 0)
+			(effects
+				(font
+					(size 1.27 1.27)
+				)
+				(hide yes)
+			)
+		)
+		(property "Datasheet" ""
+			(at 170.18 81.28 0)
+			(effects
+				(font
+					(size 1.27 1.27)
+				)
+				(hide yes)
+			)
+		)
+		(property "Description" ""
+			(at 170.18 81.28 0)
+			(effects
+				(font
+					(size 1.27 1.27)
+				)
+				(hide yes)
+			)
+		)
+		(instances
+			(project ""
+				(path "/c3e72120-9841-465e-b023-1513113688f5"
+					(reference "#G1")
+					(unit 1)
+				)
+			)
+		)
+	)
+	(symbol
 		(lib_id "power:PWR_FLAG")
 		(at 71.12 74.93 270)
@@
 		)
 	)
+	(embedded_fonts no)
 )
